Commit message: Update turtlebot3_burger_with_realsense.urdf.xacro

File: src/turtlebot3_description_custom/urdf/turtlebot3_burger_with_realsense.urdf.xacro (robot description, xacro)
@@ -1,18 +1,14 @@
 <?xml version="1.0"?>
 <robot name="turtlebot3_burger_with_realsense" xmlns:xacro="http://ros.org/wiki/xacro">
-  <!-- Include default TurtleBot3 Burger -->
   <xacro:include filename="$(find turtlebot3_description)/urdf/turtlebot3_burger.urdf.xacro"/>
   <xacro:property name="camera_height" value="0.105"/>
-  <!-- Define gray material globally -->
   <material name="gray">
     <color rgba="0.5 0.5 0.5 1.0"/>
   </material>
-  <!-- Depth Camera Joint -->
   <joint name="realsense_joint" type="fixed">
     <parent link="base_link"/>
-    <child link="realsense_link"/>
+    <child  link="realsense_link"/>
     <origin xyz="0.013 0 ${camera_height}" rpy="0 0 0"/>
   </joint>
-  <!-- Depth Camera Link -->
   <link name="realsense_link">
     <visual>
@@ -26,5 +22,5 @@
       <origin xyz="0 0 0" rpy="0 0 0"/>
       <geometry>
-        <box size="0.0 0.0 0.0"/>
+        <box size="0 0 0"/>
       </geometry>
     </collision>
@@ -35,5 +31,11 @@
     </inertial>
   </link>
-  <!-- Gazebo Plugin: RGB-D Camera -->
+  <link name="realsense_link_optical"/>
+  <joint name="realsense_optical_joint" type="fixed">
+    <parent link="realsense_link"/>
+    <child  link="realsense_link_optical"/>
+    <!-- -90° about X then -90° about Z -->
+    <origin xyz="0 0 0" rpy="-1.5708 0 -1.5708"/>
+  </joint>
   <gazebo reference="realsense_link">
     <sensor name="depth_camera" type="depth">
@@ -57,4 +59,5 @@
         <alwaysOn>true</alwaysOn>
         <updateRate>30.0</updateRate>
+        <!-- topic roots -->
         <cameraName>camera</cameraName>
         <imageTopicName>image_raw</imageTopicName>
@@ -62,5 +65,6 @@
         <cameraInfoTopicName>camera_info</cameraInfoTopicName>
         <depthCameraInfoTopicName>depth/camera_info</depthCameraInfoTopicName>
-        <frameName>realsense_link</frameName>
+        <!-- publish images in the optical frame -->
+        <frameName>realsense_link_optical</frameName>
       </plugin>
     </sensor>
